File: boards/TestBoard20/TestBoard20.kicad_sch (KiCad schematic)
At the start: 28 parts, among them J1 Conn_01x04, J10 Conn_01x02, J11 Conn_01x02, J12 Conn_01x20, J13 Conn_01x20, J14 Conn_01x20, J15 Conn_01x20, J2 Conn_01x04, J4 Conn_01x02, J6 Conn_01x20, J7 Conn_01x20, J8 Conn_01x20, J9 Conn_01x20, U1 MCP23017_SS, U2 MCP23017_SS, U3 MCP23017_SS, U4 MCP23017_SS, U5 MCP23017_SS

Commit message: Use a cheaper 20P connector, with more stock. Area for QRCode must be 8x8mm, not 7x7mm
Parts:
- J12, J13, J14, J15, J6, J7, J8, J9: LCSC C2834232 -> C19267987
Changed lines of the file:
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@@
 			)
 		)
-		(property "LCSC" "C2834232"
+		(property "LCSC" "C19267987"
 			(at 166.37 148.59 90)
 			(effects
@@
 			)
 		)
-		(property "LCSC" "C2834232"
+		(property "LCSC" "C19267987"
 			(at 113.03 166.37 90)
 			(effects
@@
 			)
 		)
-		(property "LCSC" "C2834232"
+		(property "LCSC" "C19267987"
 			(at 115.57 148.59 90)
 			(effects
@@
 			)
 		)
-		(property "LCSC" "C2834232"
+		(property "LCSC" "C19267987"
 			(at 217.17 148.59 90)
 			(effects
@@
 			)
 		)
-		(property "LCSC" "C2834232"
+		(property "LCSC" "C19267987"
 			(at 64.77 148.59 90)
 			(effects
@@
 			)
 		)
-		(property "LCSC" "C2834232"
+		(property "LCSC" "C19267987"
 			(at 62.23 166.37 90)
 			(effects
@@
 			)
 		)
-		(property "LCSC" "C2834232"
+		(property "LCSC" "C19267987"
 			(at 214.63 166.37 90)
 			(effects
@@
 			)
 		)
-		(property "LCSC" "C2834232"
+		(property "LCSC" "C19267987"
 			(at 163.83 166.37 90)
 			(effects
