File: lib/DECAP_LED/DECAP_LED.kicad_pcb (KiCad board)
At the start: 2 copper layers, 3 parts

Commit message: Set value of decap
Parts:
- DECAP.C: value (none) -> 0.1u
Changed lines of the file:
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@@
 			)
 		)
-		(property "Value" ""
+		(property "Value" "0.1u"
 			(at 0 1.16 90)
 			(layer "F.Fab")
