File: lib/DECAP_LED/DECAP_LED_flipped.kicad_pcb (KiCad board)
At the start: 2 copper layers, 3 parts

Commit message: Set value of decap
Parts:
- DECAP.C: value (none) -> 0.1u
Connections:
- DECAP.C pad 1: VDD -> GND
- DECAP.C pad 2: GND -> VDD
Changed lines of the file:
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@@
 			)
 		)
-		(property "Value" ""
+		(property "Value" "0.1u"
 			(at 0 1.16 90)
 			(layer "F.Fab")
@@
 			(layers "F.Cu" "F.Mask" "F.Paste")
 			(roundrect_rratio 0.25)
-			(net 2 "VDD")
+			(net 1 "GND")
 			(pinfunction "pin1")
 			(pintype "inout")
@@
 			(layers "F.Cu" "F.Mask" "F.Paste")
 			(roundrect_rratio 0.25)
-			(net 1 "GND")
+			(net 2 "VDD")
 			(pinfunction "pin2")
 			(pintype "inout")
@@
 	)
 	(segment
+		(start 1.751 2.681)
+		(end 1.751 3.899)
+		(width 0.2)
+		(layer "F.Cu")
+		(net 1)
+	)
+	(segment
+		(start -0.1 4)
+		(end 0.5 4)
+		(width 0.2)
+		(layer "F.Cu")
+		(net 1)
+	)
+	(segment
+		(start 0.5 4)
+		(end 1.482 4)
+		(width 0.2)
+		(layer "F.Cu")
+		(net 1)
+	)
+	(segment
+		(start 1.55 2.48)
+		(end 1.751 2.681)
+		(width 0.2)
+		(layer "F.Cu")
+		(net 1)
+	)
+	(segment
+		(start 1.65 4)
+		(end 2.1 4)
+		(width 0.2)
+		(layer "F.Cu")
+		(net 1)
+	)
+	(segment
+		(start 1.751 3.899)
+		(end 1.65 4)
+		(width 0.2)
+		(layer "F.Cu")
+		(net 1)
+	)
+	(segment
+		(start 1.482 4)
+		(end 1.65 4)
+		(width 0.2)
+		(layer "F.Cu")
+		(net 1)
+	)
+	(segment
 		(start 0.5 0)
 		(end 1.533 0)
 		(width 0.2)
 		(layer "F.Cu")
-		(net 1)
+		(net 2)
 	)
 	(segment
@@
 		(width 0.2)
 		(layer "F.Cu")
-		(net 1)
+		(net 2)
 	)
 	(segment
@@
 		(width 0.2)
 		(layer "F.Cu")
-		(net 1)
+		(net 2)
 	)
 	(segment
@@
 		(width 0.2)
 		(layer "F.Cu")
-		(net 1)
+		(net 2)
 	)
 	(segment
@@
 		(width 0.2)
 		(layer "F.Cu")
-		(net 1)
+		(net 2)
 	)
 	(segment
@@
 		(width 0.2)
 		(layer "F.Cu")
-		(net 1)
-	)
-	(segment
-		(start 1.751 2.681)
-		(end 1.751 3.899)
-		(width 0.2)
-		(layer "F.Cu")
-		(net 2)
-	)
-	(segment
-		(start -0.1 4)
-		(end 0.5 4)
-		(width 0.2)
-		(layer "F.Cu")
-		(net 2)
-	)
-	(segment
-		(start 0.5 4)
-		(end 1.482 4)
-		(width 0.2)
-		(layer "F.Cu")
-		(net 2)
-	)
-	(segment
-		(start 1.55 2.48)
-		(end 1.751 2.681)
-		(width 0.2)
-		(layer "F.Cu")
-		(net 2)
-	)
-	(segment
-		(start 1.65 4)
-		(end 2.1 4)
-		(width 0.2)
-		(layer "F.Cu")
-		(net 2)
-	)
-	(segment
-		(start 1.751 3.899)
-		(end 1.65 4)
-		(width 0.2)
-		(layer "F.Cu")
-		(net 2)
-	)
-	(segment
-		(start 1.482 4)
-		(end 1.65 4)
-		(width 0.2)
-		(layer "F.Cu")

Commit message: It seems I hadn't committed DECAP_LED_flipped.kicad_pcb
Connections:
- DECAP.C pad 1: GND -> VDD
- DECAP.C pad 2: VDD -> GND
Changed lines of the file:
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@@
 			(layers "F.Cu" "F.Mask" "F.Paste")
 			(roundrect_rratio 0.25)
-			(net 1 "GND")
+			(net 2 "VDD")
 			(pinfunction "pin1")
 			(pintype "inout")
@@
 			(layers "F.Cu" "F.Mask" "F.Paste")
 			(roundrect_rratio 0.25)
-			(net 2 "VDD")
+			(net 1 "GND")
 			(pinfunction "pin2")
 			(pintype "inout")
@@
 	)
 	(segment
+		(start 0.5 0)
+		(end 1.533 0)
+		(width 0.2)
+		(layer "F.Cu")
+		(net 1)
+	)
+	(segment
+		(start 1.76 1.31)
+		(end 1.76 0)
+		(width 0.2)
+		(layer "F.Cu")
+		(net 1)
+	)
+	(segment
+		(start 1.76 0)
+		(end 2.1 0)
+		(width 0.2)
+		(layer "F.Cu")
+		(net 1)
+	)
+	(segment
+		(start 1.533 0)
+		(end 1.76 0)
+		(width 0.2)
+		(layer "F.Cu")
+		(net 1)
+	)
+	(segment
+		(start -0.1 0)
+		(end 0.5 0)
+		(width 0.2)
+		(layer "F.Cu")
+		(net 1)
+	)
+	(segment
+		(start 1.55 1.52)
+		(end 1.76 1.31)
+		(width 0.2)
+		(layer "F.Cu")
+		(net 1)
+	)
+	(segment
 		(start 1.751 2.681)
 		(end 1.751 3.899)
 		(width 0.2)
 		(layer "F.Cu")
-		(net 1)
+		(net 2)
 	)
 	(segment
@@
 		(width 0.2)
 		(layer "F.Cu")
-		(net 1)
+		(net 2)
 	)
 	(segment
@@
 		(width 0.2)
 		(layer "F.Cu")
-		(net 1)
+		(net 2)
 	)
 	(segment
@@
 		(width 0.2)
 		(layer "F.Cu")
-		(net 1)
+		(net 2)
 	)
 	(segment
@@
 		(width 0.2)
 		(layer "F.Cu")
-		(net 1)
+		(net 2)
 	)
 	(segment
@@
 		(width 0.2)
 		(layer "F.Cu")
-		(net 1)
+		(net 2)
 	)
 	(segment
@@
 		(width 0.2)
 		(layer "F.Cu")
-		(net 1)
-	)
-	(segment
-		(start 0.5 0)
-		(end 1.533 0)
-		(width 0.2)
-		(layer "F.Cu")
-		(net 2)
-	)
-	(segment
-		(start 1.76 1.31)
-		(end 1.76 0)
-		(width 0.2)
-		(layer "F.Cu")
-		(net 2)
-	)
-	(segment
-		(start 1.76 0)
-		(end 2.1 0)
-		(width 0.2)
-		(layer "F.Cu")
-		(net 2)
-	)
-	(segment
-		(start 1.533 0)
-		(end 1.76 0)
-		(width 0.2)
-		(layer "F.Cu")
-		(net 2)
-	)
-	(segment
-		(start -0.1 0)
-		(end 0.5 0)
-		(width 0.2)
-		(layer "F.Cu")
-		(net 2)
-	)
-	(segment
-		(start 1.55 1.52)
-		(end 1.76 1.31)
-		(width 0.2)
-		(layer "F.Cu")
